File: schematic/vrx.sch (EAGLE design)
At the start: 20 parts, among them IC1 4066N, SW1 EC12E_SW, X1 22-23-2021, X2 22-23-2021, X3 22-23-2021, X4 22-23-2051, X5 22-23-2051, X6 22-23-2041

Commit message: clean garbage
Parts:
- removed JP1: (no value), pinhead:PINHD-1X4
- removed X2, X3: 22-23-2021, con-molex:22-23-2021
- removed X6: 22-23-2041, con-molex:22-23-2041
- added U$3: DISPLAY-OLED-128X64-I2C, diy-modules:DISPLAY-OLED-128X64-I2C
- added X7: 22-23-2031, con-molex:22-23-2031
- R5, R6, R7: value 170k -> 1K
- R8, R9: value 170k -> 10K
Connections:
- removed net 3.3V: JP1.2
- removed net N$1: IC1A.B, IC1B.B, X6-1.S
- removed net N$2: IC1C.B, IC1D.B, X6-3.S
- removed net N$5: IC1A.A, X2-2.S
- removed net N$6: IC1B.A, X2-1.S
- removed net N$7: IC1C.A, X3-2.S
- removed net N$8: IC1D.A, X3-1.S
- new net BASE_BAND1: IC1A.A, X7-1.S
- new net BASE_BAND2: IC1B.A, X7-2.S
- new net BASE_BAND_OUT: IC1A.B, IC1B.B, X7-3.S
- new net TUN1_SEL: IC1A.C, U$1.PB12
- new net TUN2_SEL: IC1B.C, U$1.PB13
- net GND: now also U$3.GND; no longer JP1.1, X6-2.S, X6-4.S
- net I2C2_SCL: now also U$3.SCL; no longer JP1.3
- net I2C2_SDA: now also U$3.SDA; no longer JP1.4
- net PB3: no longer IC1A.C, IC1C.C
- net PB7: no longer IC1B.C, IC1D.C
- net VDD: now also U$3.VCC
Other:
- moved on the sheet: X4-1, X4-2, X4-3, X4-4, X4-5, X5-1, X5-2, X5-3, X5-4, X5-5
